File: lighthouse.kicad_pcb (KiCad board)
At the start: 2 copper layers, 0 parts

Commit message: Schematic and PCB
Parts:
- added C1: 2u2 35V, Capacitor_SMD:C_0603_1608Metric_Pad1.08x0.95mm_HandSolder, B.Cu at (138.0, 91.7)
- added C10: 10n, Capacitor_SMD:C_0603_1608Metric_Pad1.08x0.95mm_HandSolder, B.Cu at (153.4, 113.8)
- added C11: 1u, Capacitor_SMD:C_0603_1608Metric_Pad1.08x0.95mm_HandSolder, B.Cu at (147.4, 121.9)
- added C12: 100n, Capacitor_SMD:C_0603_1608Metric_Pad1.08x0.95mm_HandSolder, B.Cu at (147.9, 120.5)
- added C2: 100n, Capacitor_SMD:C_0603_1608Metric_Pad1.08x0.95mm_HandSolder, B.Cu at (154.5, 111.1)
- added C3: 22u, Capacitor_SMD:C_0805_2012Metric_Pad1.18x1.45mm_HandSolder, B.Cu at (136.2, 94.4)
- added C4: 100n, Capacitor_SMD:C_0603_1608Metric_Pad1.08x0.95mm_HandSolder, B.Cu at (159.1, 120.0)
- added C6: 10u, Capacitor_SMD:C_0805_2012Metric_Pad1.18x1.45mm_HandSolder, B.Cu at (145.5, 119.2)
- added C7: 100n, Capacitor_SMD:C_0603_1608Metric_Pad1.08x0.95mm_HandSolder, B.Cu at (153.6, 122.9)
- added C8: 100n, Capacitor_SMD:C_0603_1608Metric_Pad1.08x0.95mm_HandSolder, B.Cu at (149.5, 114.8)
- added C9: 1u, Capacitor_SMD:C_0603_1608Metric_Pad1.08x0.95mm_HandSolder, B.Cu at (154.0, 112.5)
- added D1: LED, LED_THT:LED_D5.0mm_Horizontal_O3.81mm_Z3.0mm, F.Cu at (158.7, 109.8)
- added D10: ESD5Zxx, Diode_SMD:D_SOD-523, B.Cu at (163.8, 121.8)
- added D11: ESD5Zxx, Diode_SMD:D_SOD-523, B.Cu at (162.7, 122.9)
- added D12: ESD5Zxx, Diode_SMD:D_SOD-523, B.Cu at (173.0, 120.2)
- added D13: TVS (P6SMB16CA), Diode_SMD:D_SMB_Handsoldering, B.Cu at (146.4, 82.8)
- added D2: LED, LED_THT:LED_D5.0mm_Horizontal_O3.81mm_Z3.0mm, F.Cu at (152.2, 106.0)
- added D3: LED, LED_THT:LED_D5.0mm_Horizontal_O3.81mm_Z3.0mm, F.Cu at (150.2, 98.7)
- added D4: LED, LED_THT:LED_D5.0mm_Horizontal_O3.81mm_Z3.0mm, F.Cu at (154.0, 92.2)
- added D5: LED, LED_THT:LED_D5.0mm_Horizontal_O3.81mm_Z3.0mm, F.Cu at (161.3, 90.2)
- added D6: LED, LED_THT:LED_D5.0mm_Horizontal_O3.81mm_Z3.0mm, F.Cu at (167.8, 94.0)
- added D7: LED, LED_THT:LED_D5.0mm_Horizontal_O3.81mm_Z3.0mm, F.Cu at (169.8, 101.3)
- added D8: LED, LED_THT:LED_D5.0mm_Horizontal_O3.81mm_Z3.0mm, F.Cu at (166.0, 107.8)
- added D9: ESD5Zxx, Diode_SMD:D_SOD-523, B.Cu at (163.8, 115.0)
- added H1: MountingHole, MountingHole:MountingHole_3.2mm_M3_ISO14580, F.Cu at (156.0, 100.0)
- added H2: MountingHole, MountingHole:MountingHole_3.2mm_M3_ISO14580, F.Cu at (164.0, 100.0)
- added J1: PB4, Connector_PinHeader_2.54mm:PinHeader_1x01_P2.54mm_Vertical, B.Cu at (139.2, 108.8)
- added J10: Input, Connector_Molex:Molex_PicoBlade_53047-0210_1x02_P1.25mm_Vertical, B.Cu at (140.6, 87.0)
- added J11: I²C, Connector_Molex:Molex_PicoBlade_53047-0410_1x04_P1.25mm_Vertical, B.Cu at (180.8, 111.9)
- added J12: Photoresistor, Connector_Molex:Molex_PicoBlade_53047-0210_1x02_P1.25mm_Vertical, B.Cu at (159.4, 125.0)
- added J2: PB5, Connector_PinHeader_2.54mm:PinHeader_1x01_P2.54mm_Vertical, B.Cu at (139.2, 104.5)
- added J3: PB6, Connector_PinHeader_2.54mm:PinHeader_1x01_P2.54mm_Vertical, B.Cu at (143.0, 108.8)
- added J4: PB7, Connector_PinHeader_2.54mm:PinHeader_1x01_P2.54mm_Vertical, B.Cu at (143.0, 104.5)
- added J5: SWD, Connector_PinHeader_1.27mm:PinHeader_2x05_P1.27mm_Vertical_SMD, B.Cu at (167.6, 119.0)
- added J8: PA12, Connector_PinHeader_2.54mm:PinHeader_1x01_P2.54mm_Vertical, B.Cu at (142.5, 117.5)
- added L1: 10u, Inductor_SMD:L_1210_3225Metric, B.Cu at (137.8, 98.2)
- added Q1: BC846, Package_TO_SOT_SMD:SOT-23, B.Cu at (158.8, 114.8)
- added Q2: BC846, Package_TO_SOT_SMD:SOT-23, B.Cu at (148.5, 109.6)
- added Q3: BC846, Package_TO_SOT_SMD:SOT-23, B.Cu at (145.2, 98.8)
- added Q4: BC846, Package_TO_SOT_SMD:SOT-23, B.Cu at (150.6, 88.8)
- added Q5: BC846, Package_TO_SOT_SMD:SOT-23, B.Cu at (161.2, 85.2)
- added Q6: BC846, Package_TO_SOT_SMD:SOT-23, B.Cu at (171.2, 90.6)
- added Q7: BC846, Package_TO_SOT_SMD:SOT-23, B.Cu at (174.8, 101.2)
- added Q8: BC846, Package_TO_SOT_SMD:SOT-23, B.Cu at (169.4, 111.2)
- added R1: 4k7 1%, Resistor_SMD:R_0603_1608Metric_Pad0.98x0.95mm_HandSolder, B.Cu at (141.5, 91.4)
- added R10: R, Resistor_SMD:R_0603_1608Metric_Pad0.98x0.95mm_HandSolder, B.Cu at (142.5, 98.8)
- added R11: R, Resistor_SMD:R_0603_1608Metric_Pad0.98x0.95mm_HandSolder, B.Cu at (148.0, 98.8)
- added R12: R, Resistor_SMD:R_0603_1608Metric_Pad0.98x0.95mm_HandSolder, B.Cu at (148.6, 86.9)
- added R13: R, Resistor_SMD:R_0603_1608Metric_Pad0.98x0.95mm_HandSolder, B.Cu at (152.5, 90.8)
- added R14: R, Resistor_SMD:R_0603_1608Metric_Pad0.98x0.95mm_HandSolder, B.Cu at (161.2, 82.5)
- added R15: R, Resistor_SMD:R_0603_1608Metric_Pad0.98x0.95mm_HandSolder, B.Cu at (161.2, 88.0)
- added R16: R, Resistor_SMD:R_0603_1608Metric_Pad0.98x0.95mm_HandSolder, B.Cu at (173.1, 88.6)
- added R17: R, Resistor_SMD:R_0603_1608Metric_Pad0.98x0.95mm_HandSolder, B.Cu at (169.2, 92.5)
- added R18: R, Resistor_SMD:R_0603_1608Metric_Pad0.98x0.95mm_HandSolder, B.Cu at (177.5, 101.2)
- added R19: R, Resistor_SMD:R_0603_1608Metric_Pad0.98x0.95mm_HandSolder, B.Cu at (172.0, 101.2)
- added R2: 1k5 1%, Resistor_SMD:R_0603_1608Metric_Pad0.98x0.95mm_HandSolder, B.Cu at (143.2, 91.4)
- added R20: R, Resistor_SMD:R_0603_1608Metric_Pad0.98x0.95mm_HandSolder, B.Cu at (171.4, 113.1)
- added R21: R, Resistor_SMD:R_0603_1608Metric_Pad0.98x0.95mm_HandSolder, B.Cu at (167.5, 109.2)
- added R3: R, Resistor_SMD:R_0603_1608Metric_Pad0.98x0.95mm_HandSolder, B.Cu at (158.8, 117.5)
- added R4: R, Resistor_SMD:R_0603_1608Metric_Pad0.98x0.95mm_HandSolder, B.Cu at (158.8, 112.0)
- added R5: R, Resistor_SMD:R_0603_1608Metric_Pad0.98x0.95mm_HandSolder, B.Cu at (146.6, 111.6)
- added R6: 2k2, Resistor_SMD:R_0603_1608Metric_Pad0.98x0.95mm_HandSolder, B.Cu at (178.5, 116.5)
- added R7: 100k, Resistor_SMD:R_0603_1608Metric_Pad0.98x0.95mm_HandSolder, B.Cu at (159.0, 121.5)
- added R8: 2k2, Resistor_SMD:R_0603_1608Metric_Pad0.98x0.95mm_HandSolder, B.Cu at (179.8, 114.8)
- added R9: R, Resistor_SMD:R_0603_1608Metric_Pad0.98x0.95mm_HandSolder, B.Cu at (150.5, 107.6)
- added U1: TPS62175DQC, Package_SON:WSON-10-1EP_2x3mm_P0.5mm_EP0.84x2.4mm_ThermalVias, B.Cu at (139.8, 94.7)
- added U2: STM32L072KBUx, Package_DFN_QFN:QFN-32-1EP_5x5mm_P0.5mm_EP3.45x3.45mm, B.Cu at (152.6, 118.0)
Routing:
- net +3V3: track 0.00 -> 198.2 mm, vias 0 -> 7
- net /LED4: track 0.00 -> 45.8 mm, vias 0 -> 2
- net /LED5: track 0.00 -> 44.2 mm, vias 0 -> 2
- net /LED3: track 0.00 -> 41.9 mm, vias 0 -> 2
- net /I²C1_SDA: track 0.00 -> 36.9 mm, vias 0 -> 2
- net GND: track 0.00 -> 36.8 mm, vias 0 -> 119
- net /I²C1_SCL: track 0.00 -> 35.6 mm, vias 0 -> 2
- net /LED6: track 0.00 -> 35.2 mm, vias 0 -> 2
- net /LED2: track 0.00 -> 29.9 mm, vias 0 -> 2
- net /~{RST}: track 0.00 -> 28.2 mm, vias 0 -> 4
- net /SWCLK: track 0.00 -> 27.0 mm, vias 0 -> 2
- net /LED7: track 0.00 -> 22.0 mm, vias 0 -> 2
- net /SWDIO: track 0.00 -> 19.4 mm, vias 0 -> 2
- net Net-(J2-Pin_1): track 0.00 -> 18.7 mm
- net /LED1: track 0.00 -> 17.7 mm, vias 0 -> 2
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- added copper zone on B.Cu, net GND
- added copper zone on F.Cu, net GND
Other:
- board outline added: 54 x 54 mm
- board text added: "lighthouse v1.0 2024-06 by MG-5"
